File: Kicad_Files/WarpESC.kicad_sch (KiCad schematic)
At the start: 94 parts, among them IC1 STM32F303RBT6XXXTR, IC2 SIC634CD-T1-GE3, IC3 SIC634CD-T1-GE3, IC4 SIC634CD-T1-GE3, IC5 SIC634CD-T1-GE3, IC6 SIC634CD-T1-GE3, IC7 SIC634CD-T1-GE3, J1 USB_B_Micro, J10 Conn_01x01_Female, J11 VV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

Commit message: Add files via upload
Parts:
- removed C5: 150uF, symbol Device:C_Small
- C4: value 150uF -> 470uF
- J10, J11, J12, J13, J14, J15, J16, J17, J2, J4, J5, J6, J7, J8, J9, JP1: now left out of the parts list
Other:
- note added: "externally connected"
- moved on the sheet: C1, C10, C11, C12, C13, C14, C15, C16, C17, C18, C19, C2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
